Commit message: Use real PH42 interface and add RealSense D435 mount
- J6 adapter flange: 8x M3 and 4x dowel holes at the positions measured
  from the PH42-020-S300-R STEP, plus a centring boss into the horn recess;
  real PH42 model replaces the envelope (parts/PH42-020-S300-R.stp)
- RealSense D435/D435i eye-in-hand: camera on a flat bracket plate, low on
  the base plate and 0.5 mm from the front plate; front-plate tabs moved
  to x = +/-50, base plate extended to y = 42
- URDF: camera_link and camera_depth_optical_frame at the D435 depth origin;
  STLs and URDF meshes regenerated

Co-Authored-By: Claude Opus 5.5 <noreply@anthropic.com>

File: gripper_mx64_ph42.urdf (robot description, URDF)
Before this commit: robot gripper_mx64_ph42, 8 links, 7 joints
Links:
- added link camera_depth_optical_frame
- added link camera_link
- link gripper_base_link: mass 0.791289 -> 0.905847; geometry collision mesh filename=urdf_meshes/back_plate.stl scale=0.001 0.001 0.001; collision mesh filename=urdf_meshes/base_plate.stl scale=0.001 0.001 0.001
Joints:
- added joint camera_depth_optical_joint: type fixed, parent camera_link, child camera_depth_optical_frame, origin xyz=0 0 0 rpy=-1.5708 0 -1.5708
- added joint camera_joint: type fixed, parent gripper_base_link, child camera_link, origin xyz=0.0175 0.016 0.03685 rpy=0 -1.5708 -1.5708
